File: Wiring_Diagram/Wiring_Diagram.kicad_pcb (KiCad board)
At the start: 2 copper layers, 9 parts, among them SW1 SW_Push, SW2 SW_Push, SW3 SW_Push, SW4 SW_Push

Commit message: added README
Parts:
- R1: moved to B.Cu
- moved D4 81.5 mm to (122.0, 92.4), turned to 90 degrees
- moved D3 66.0 mm to (102.8, 92.4), turned to 90 degrees
- moved D2 53.7 mm to (83.7, 92.4), turned to 90 degrees
- moved D1 46.8 mm to (64.8, 92.4), turned to 90 degrees
- moved R1 44.3 mm to (75.4, 103.2), turned to 180 degrees
Routing:
- net Net-(D1-K): track 0.00 -> 11.4 mm
- net Net-(D2-K): track 0.00 -> 11.3 mm
- net Net-(D4-K): track 0.00 -> 11.2 mm
- net Net-(D3-K): track 0.00 -> 11.1 mm
- net Net-(R1-Pad2): track 0.00 -> 4.51 mm
- added copper zone on F.Cu, net +9V
- added copper zone on B.Cu, net GND
Other:
- board outline added: 73.7 x 15.5 mm
